Commit message: Update for 6-dof planning, better planning scenes, better urdf

File: urdf/franka_panda/panda.urdf (robot description, URDF)
Before this commit: robot panda, 15 links, 14 joints
Links:
- removed link end_effector_frame
- removed link world
- added link panda_grasptarget, mass 0.0
- link panda_hand: mass 0.73 -> .81; geometry collision mesh filename=package://meshes/collision/hand.obj; visual mesh filename=package://meshes/visual/hand.obj
- link panda_leftfinger: geometry collision mesh filename=package://meshes/collision/finger.obj; visual mesh filename=package://meshes/visual/finger.obj
- link panda_link0: mass 2.92 -> 2.9; geometry collision mesh filename=package://meshes/collision/link0.obj; visual mesh filename=package://meshes/collision/link0.obj
- link panda_link1: mass 2.74 -> 2.7; geometry collision mesh filename=package://meshes/collision/link1.obj; visual mesh filename=package://meshes/visual/link1.obj
- link panda_link2: mass 2.74 -> 2.73; geometry collision mesh filename=package://meshes/collision/link2.obj; visual mesh filename=package://meshes/visual/link2.obj
- link panda_link3: mass 2.38 -> 2.04; geometry collision mesh filename=package://meshes/collision/link3.obj; visual mesh filename=package://meshes/visual/link3.obj
- link panda_link4: mass 2.38 -> 2.08; geometry collision mesh filename=package://meshes/collision/link4.obj; visual mesh filename=package://meshes/visual/link4.obj
- link panda_link5: mass 2.74 -> 3; geometry collision mesh filename=package://meshes/collision/link5.obj; visual mesh filename=package://meshes/visual/link5.obj
- link panda_link6: mass 1.55 -> 1.3; geometry collision mesh filename=package://meshes/collision/link6.obj; visual mesh filename=package://meshes/visual/link6.obj
- link panda_link7: mass 0.54 -> .2; geometry collision mesh filename=package://meshes/collision/link7.obj; visual mesh filename=package://meshes/collision/link7.obj
- link panda_link8: mass None -> 0.0
- link panda_rightfinger: geometry collision mesh filename=package://meshes/collision/finger.obj; visual mesh filename=package://meshes/visual/finger.obj
Joints:
- removed joint end_effector_frame_fixed_joint
- removed joint panda_joint_world
- added joint panda_grasptarget_hand: type fixed, parent panda_hand, child panda_grasptarget, origin xyz=0 0 0.105 rpy=0 0 0
- joint panda_finger_joint1: limit lower=-0.001 upper=0.04 effort=20 velocity=0.3 -> lower=0.0 upper=0.04 effort=20 velocity=0.2
- joint panda_finger_joint2: limit lower=-0.001 upper=0.04 effort=20 velocity=0.3 -> lower=0.0 upper=0.04 effort=20 velocity=0.2; mimic (none) -> joint=panda_finger_joint1
- joint panda_joint1: limit lower=-2.8973 upper=2.8973 effort=87 velocity=2.1750 -> lower=-2.9671 upper=2.9671 effort=87 velocity=2.1750
- joint panda_joint2: limit lower=-1.7628 upper=1.7628 effort=87 velocity=2.1750 -> lower=-1.8326 upper=1.8326 effort=87 velocity=2.1750
- joint panda_joint3: limit lower=-2.8973 upper=2.8973 effort=87 velocity=2.1750 -> lower=-2.9671 upper=2.9671 effort=87 velocity=2.1750
- joint panda_joint4: limit lower=-3.0718 upper=0.0698 effort=87 velocity=2.1750 -> lower=-3.1416 upper=0.0 effort=87 velocity=2.1750
- joint panda_joint5: limit lower=-2.8973 upper=2.8973 effort=12 velocity=2.6100 -> lower=-2.9671 upper=2.9671 effort=12 velocity=2.6100
- joint panda_joint6: limit lower=-0.0175 upper=3.7525 effort=12 velocity=2.6100 -> lower=-0.0873 upper=3.8223 effort=12 velocity=2.6100
- joint panda_joint7: limit lower=-2.8973 upper=2.8973 effort=12 velocity=2.6100 -> lower=-2.9671 upper=2.9671 effort=12 velocity=2.6100

File: urdf/panda_hand/panda.urdf (robot description, URDF)
Before this commit: robot panda_hand, 8 links, 7 joints
Links:
- added link base_frame, mass 0
- added link right_gripper, mass 0.01
Joints:
- added joint base_frame_panda_hand: type fixed, parent base_frame, child panda_hand, origin xyz=0 0 0 rpy=0 0 -0.78539816337, axis 1 0 0
- added joint right_gripper: type fixed, parent base3, child right_gripper, origin xyz=0 0 0.1 rpy=0 0 2.35619449019, axis 0 0 1
- joint base3_base_link: child panda_hand -> base_frame
